Commit message: Upate launch files and model file for inconsistant of xacro label

File: icl_ur5_setup_description/robots/ur5_robotiq_140_joint_limited.xacro (robot description, xacro)
@@ -1,4 +1,4 @@
 <?xml version="1.0"?>
-<robot xmlns:xacro="http://ros.org/wiki/xacro" name="ur5_gripper">
+<robot xmlns:xacro="http://wiki.ros.org/xacro" name="ur5_gripper">
   <!-- include macros for UR5 and the Robotiq eef model -->
   <xacro:include filename="$(find ur_description)/urdf/common.gazebo.xacro" />

File: icl_ur5_setup_description/robots/ur5_robotiq_140_joint_limited_kinect2.xacro (robot description, xacro)
@@ -1,4 +1,4 @@
 <?xml version="1.0"?>
-<robot xmlns:xacro="http://ros.org/wiki/xacro" name="ur5_gripper">
+<robot xmlns:xacro="http://wiki.ros.org/xacro" name="ur5_gripper">
   <!-- include macros for UR5 and the Robotiq eef model -->
   <xacro:include filename="$(find ur_description)/urdf/common.gazebo.xacro" />

File: icl_ur5_setup_description/urdf/robotiq_arg2f.xacro (robot description, xacro)
@@ -1,4 +1,4 @@
 <?xml version="1.0"?>
-<robot xmlns:xacro="http://ros.org/wiki/xacro">
+<robot xmlns:xacro="http://wiki.ros.org/xacro">
   <!--xacro:include filename="$(find icl_phri_ur5_robotiq_arg140_description)/urdf/robotiq_arg2f_finger_tips.xacro" /-->
   <xacro:macro name="robotiq_arg2f_base_link" params="prefix">

File: icl_ur5_setup_description/urdf/robotiq_arg2f_140_model_macro.xacro (robot description, xacro)
@@ -1,4 +1,4 @@
 <?xml version="1.0"?>
-<robot xmlns:xacro="http://ros.org/wiki/xacro">
+<robot xmlns:xacro="http://wiki.ros.org/xacro">
   <xacro:include filename="$(find icl_ur5_setup_description)/urdf/robotiq_arg2f_transmission.xacro" />
   <xacro:macro name="outer_knuckle" params="prefix fingerprefix stroke">

File: icl_ur5_setup_description/urdf/robotiq_arg2f_transmission.xacro (robot description, xacro)
@@ -1,4 +1,4 @@
 <?xml version="1.0"?>
-<robot xmlns:xacro="http://ros.org/wiki/xacro">
+<robot xmlns:xacro="http://wiki.ros.org/xacro">
   <xacro:macro name="robotiq_arg2f_transmission" params="prefix hw_interface">
     <transmission name="${prefix}finger_joint_trans">

File: icl_ur5_setup_description/urdf/robotiq_fts300.urdf.xacro (robot description, xacro)
@@ -1,4 +1,4 @@
 <?xml version="1.0"?>
-<robot xmlns:xacro="http://ros.org/wiki/xacro" name="robotiq_fts150">
+<robot xmlns:xacro="http://wiki.ros.org/xacro" name="robotiq_fts150">
     <xacro:macro name="robotiq_fts150" params="parent prefix *origin">
         <!-- mount the fts to the robot -->

File: icl_ur5_setup_description/urdf/sensors/common.xacro (robot description, xacro)
@@ -1,4 +1,4 @@
 <?xml version="1.0"?>
-<robot xmlns:xacro="http://www.ros.org/wiki/xacro">
+<robot xmlns:xacro="http://wiki.ros.org/xacro">
   <xacro:property name="M_PI" value="3.1415926535897931" />
   <xacro:property name="VELOCITY_LIMIT_SCALE" value="0.6" />

File: icl_ur5_setup_description/urdf/sensors/kinect2.gazebo.xacro (robot description, xacro)
@@ -1,4 +1,4 @@
 <?xml version="1.0"?>
-<robot xmlns:xacro="http://www.ros.org/wiki/xacro">
+<robot xmlns:xacro="http://wiki.ros.org/xacro">
 <xacro:macro name="kinect2_ir_gazebo_v0" params="link_name frame_name camera_name">
   <gazebo reference="${link_name}">

File: icl_ur5_setup_description/urdf/sensors/kinect2.urdf.xacro (robot description, xacro)
@@ -1,4 +1,4 @@
 <?xml version="1.0"?>
-<robot xmlns:xacro="http://www.ros.org/wiki/xacro">
+<robot xmlns:xacro="http://wiki.ros.org/xacro">
   <xacro:include filename="$(find icl_ur5_setup_description)/urdf/sensors/kinect2.gazebo.xacro" />
   <xacro:property name="ir_depth_rgb_offset_y" value="0.01"/> <!-- FIXME: what is this offset? -->
@@ -21,5 +21,5 @@
         <origin xyz="-0.102 -0.148 0" rpy="0 0 0"/>
         <geometry>
-          <mesh filename="package://pr2_description/meshes/sensors/kinect2_v0/kinect2_assembly.dae" scale="0.001 0.001 0.001" />
+          <mesh filename="package://icl_ur5_setup_description/meshes/sensors/kinect2_v0/kinect2_assembly.dae" scale="0.001 0.001 0.001" />
         </geometry>
         <material name="gray">

File: ur5_description/urdf/common.gazebo.xacro (robot description, xacro)
@@ -1,4 +1,4 @@
 <?xml version="1.0"?>
-<robot xmlns:xacro="http://ros.org/wiki/xacro">
+<robot xmlns:xacro="http://wiki.ros.org/xacro">
   <gazebo>
     <plugin name="ros_control" filename="libgazebo_ros_control.so">

File: ur5_description/urdf/ur.gazebo.xacro (robot description, xacro)
@@ -1,4 +1,4 @@
 <?xml version="1.0"?>
-<robot xmlns:xacro="http://ros.org/wiki/xacro">
+<robot xmlns:xacro="http://wiki.ros.org/xacro">
   <xacro:macro name="ur_arm_gazebo" params="prefix">
     <gazebo reference="${prefix}shoulder_link">

File: ur5_description/urdf/ur5.urdf.xacro (robot description, xacro)
@@ -1,4 +1,4 @@
 <?xml version="1.0"?>
-<robot xmlns:xacro="http://ros.org/wiki/xacro">
+<robot xmlns:xacro="http://wiki.ros.org/xacro">
   <xacro:include filename="$(find ur_description)/urdf/ur.transmission.xacro" />
   <xacro:include filename="$(find ur_description)/urdf/ur.gazebo.xacro" />

File: ur5_description/urdf/ur5_joint_limited_robot.urdf.xacro (robot description, xacro)
@@ -1,4 +1,4 @@
 <?xml version="1.0"?>
-<robot xmlns:xacro="http://ros.org/wiki/xacro"
+<robot xmlns:xacro="http://wiki.ros.org/xacro"
        name="ur5" >
   <!-- common stuff -->

File: ur5_description/urdf/ur5_robot.urdf.xacro (robot description, xacro)
@@ -1,4 +1,4 @@
 <?xml version="1.0"?>
-<robot xmlns:xacro="http://ros.org/wiki/xacro"
+<robot xmlns:xacro="http://wiki.ros.org/xacro"
        name="ur5" >
   <!-- common stuff -->
