Commit message: add model files and configuration files

File: icl_ur5_setup_description/robots/ur5_robotiq_140_joint_limited_kinect2.xacro (robot description, xacro)
@@ -6,4 +6,6 @@
   <xacro:include filename="$(find icl_ur5_setup_description)/urdf/robotiq_arg2f_140_model_macro.xacro" />
   <xacro:include filename="$(find icl_ur5_setup_description)/urdf/robotiq_fts300.urdf.xacro" />
+  <xacro:include filename="$(find icl_ur5_setup_description)/urdf/sensors/common.xacro" />
+  <xacro:include filename="$(find icl_ur5_setup_description)/urdf/sensors/kinect2.urdf.xacro" />
   <xacro:macro name="ur5_with_gripper_joint_limited" params="prefix">
     <!-- arm -->
@@ -50,4 +52,8 @@
     </joint>
     </xacro:macro>
+    <xacro:kinect2_v0 name="" parent="world" >
+      <!--origin xyz="0.4 0.0 1.2" rpy="0.0 ${pi/2} 0.0" /-->
+      <origin xyz="2 0.0 1.3" rpy="0.0 ${pi/3} ${pi}" />
+    </xacro:kinect2_v0>
   <xacro:ur5_with_gripper_joint_limited prefix=""/>
  <!-- Plugin -->

File: icl_ur5_setup_description/urdf/robotiq_arg2f_transmission.xacro (robot description, xacro)
@@ -1,9 +1,9 @@
 <?xml version="1.0"?>
 <robot xmlns:xacro="http://ros.org/wiki/xacro">
-  <xacro:macro name="robotiq_arg2f_transmission" params="prefix">
+  <xacro:macro name="robotiq_arg2f_transmission" params="prefix hw_interface">
     <transmission name="${prefix}finger_joint_trans">
       <type>transmission_interface/SimpleTransmission</type>
       <joint name="${prefix}finger_joint">
-        <hardwareInterface>PositionJointInterface</hardwareInterface>
+        <hardwareInterface>${hw_interface}</hardwareInterface>
       </joint>
       <actuator name="${prefix}finger_joint_motor">

Commit message: add rg6 model

File: icl_ur5_setup_description/robots/ur5_robotiq_140_joint_limited_kinect2.xacro (robot description, xacro)
@@ -31,9 +31,9 @@
       <child link = "${prefix}base_link" />
       <!--origin xyz="0.0 0.0 0.0" rpy="0.0 0.0 0.0" /-->
-      <origin xyz="0.0 0.0 0.7" rpy="0.0 0.0 0.0" />
+      <origin xyz="0.0 0.0 0.4" rpy="0.0 0.0 0.0" />
     </joint>
     <!--force torque sensor-->
     <xacro:robotiq_fts150 prefix="" parent="ee_link" >
-      <origin xyz="0.009 0 0 " rpy="-${pi/2} 0 -${pi/2}"/>
+      <origin xyz="0.001 0 0 " rpy="-${pi/2} 0 -${pi/2}"/>
     </xacro:robotiq_fts150>
    <!-- gripper -->
@@ -49,7 +49,7 @@
       <parent link= "${prefix}ee_link" />
       <child link = "${prefix}tool" />
-      <origin xyz=" 0.00 0.0 0.2" rpy="0.0 0.0 0.0" />
+      <origin xyz=" 0.2 0.0 0.0" rpy="0.0 0.0 0.0" />
     </joint>
-    </xacro:macro>
+  </xacro:macro>
     <xacro:kinect2_v0 name="" parent="world" >
       <!--origin xyz="0.4 0.0 1.2" rpy="0.0 ${pi/2} 0.0" /-->

File: icl_ur5_setup_description/urdf/sensors/kinect2.gazebo.xacro (robot description, xacro)
@@ -29,9 +29,11 @@
         <pointCloudTopicName>/${camera_name}/depth/points</pointCloudTopicName>
         <frameName>${frame_name}</frameName>
+        <!--pointCloudCutoff>1.5</pointCloudCutoff-->
+        <!--pointCloudCutoffMax>3.0</pointCloudCutoffMax-->
         <pointCloudCutoff>0.5</pointCloudCutoff>
         <distortionK1>0.00000001</distortionK1>
         <distortionK2>0.00000001</distortionK2>
         <distortionK3>0.00000001</distortionK3>
-        <distortionT1>0.00000001</distortionT1>
+        <distortionT1>0.00000001</distortionT1>a
         <distortionT2>0.00000001</distortionT2>
         <CxPrime>0</CxPrime>
