Commit message: add DOPE env

File: icl_ur5_setup_description/robots/kinect2_3D_object.xacro (robot description, xacro)
@@ -9,6 +9,6 @@
   <xacro:kinect2_v0 name="" parent="world" >
     <!--origin xyz="0.4 0.0 1.2" rpy="0.0 ${pi/2} 0.0" /-->
-    <!--origin xyz="1.4 0.0 0.60" rpy="0.0 ${pi/10} ${pi}" /-->
-    <origin xyz="-1.3 1.3 1.3" rpy="0.0 ${2*pi/9} ${-1*pi/4}" />
+    <origin xyz="1.0 0.0 0.6" rpy="0.0 ${pi/10} ${pi}" />
+    <!--origin xyz="-1.3 1.3 1.3" rpy="0.0 ${2*pi/9} ${-1*pi/4}" /-->
     </xacro:kinect2_v0>
     <!--joint name="ur5_ee_link-gripper_base" type="fixed">

File: icl_ur5_setup_description/robots/ur5_rg6_kinect2.xacro (robot description, xacro)
@@ -29,5 +29,6 @@
   <xacro:kinect2_v0 name="" parent="world" >
     <!--origin xyz="0.4 0.0 1.2" rpy="0.0 ${pi/2} 0.0" /-->
-    <origin xyz="1.5 0.0 1.3" rpy="0.0 ${pi/3} ${pi}" />
+    <!--origin xyz="1.5 0.0 1.3" rpy="0.0 ${pi/3} ${pi}" /-->
+    <origin xyz="-1.3 1.3 1.3" rpy="0.0 ${2*pi/9} ${-1*pi/4}" />
   </xacro:kinect2_v0>
     <!--joint name="ur5_ee_link-gripper_base" type="fixed">

File: icl_ur5_setup_description/robots/ur5_robotiq_140_joint_limited_kinect2.xacro (robot description, xacro)
@@ -19,5 +19,5 @@
     /-->
     <xacro:ur5_robot prefix="${prefix}" joint_limited="true"
-      shoulder_pan_lower_limit="${-2*pi}" shoulder_pan_upper_limit="${2*pi}"
+      shoulder_pan_lower_limit="${-pi}" shoulder_pan_upper_limit="${pi}"
       shoulder_lift_lower_limit="${-pi}" shoulder_lift_upper_limit="${pi}"
       elbow_joint_lower_limit="${-pi}" elbow_joint_upper_limit="${pi}"
@@ -54,5 +54,7 @@
     <xacro:kinect2_v0 name="" parent="world" >
       <!--origin xyz="0.4 0.0 1.2" rpy="0.0 ${pi/2} 0.0" /-->
-      <origin xyz="2 0.0 1.3" rpy="0.0 ${pi/3} ${pi}" />
+      <!--origin xyz="2 0.0 1.3" rpy="0.0 ${pi/3} ${pi}" /-->
+      <!--origin xyz="-1.3 1.3 1.3" rpy="0.0 ${2*pi/9} ${-1*pi/4}" /-->
+      <origin xyz="1.3 -1.3 1.3" rpy="0.0 ${2*pi/9} ${3*pi/4}" />
     </xacro:kinect2_v0>
   <xacro:ur5_with_gripper_joint_limited prefix=""/>
@@ -61,10 +63,10 @@
     <plugin name="gazebo_grasp_fix" filename="libgazebo_grasp_fix.so">
       <arm>
-          <arm_name>robot</arm_name>
+          <arm_name>ur5_robot</arm_name>
           <palm_link>wrist_3_link</palm_link>
           <gripper_link>left_inner_finger</gripper_link>
           <gripper_link>right_inner_finger</gripper_link>
-          <gripper_link>left_inner_knuckle</gripper_link>
-          <gripper_link>right_inner_knuckle</gripper_link>
+          <!--gripper_link>left_inner_knuckle</gripper_link>
+          <gripper_link>right_inner_knuckle</gripper_link-->
       </arm>
       <forces_angle_tolerance>120</forces_angle_tolerance>
@@ -72,5 +74,5 @@
       <grip_count_threshold>4</grip_count_threshold>
       <max_grip_count>8</max_grip_count>
-      <release_tolerance>0.05</release_tolerance>
+      <release_tolerance>0.02</release_tolerance>
       <disable_collisions_on_attach>true</disable_collisions_on_attach>
       <contact_topic>__default_topic__</contact_topic>

File: icl_ur5_setup_description/urdf/robotiq_arg2f_140_model_macro.xacro (robot description, xacro)
@@ -217,5 +217,6 @@
     <link name="${prefix}${fingerprefix}_finger_tip">
       <inertial>
-        <origin xyz="0.000299999999999317 0.0160078233491243 -0.0136945669206257" rpy="0 0 0" />
+        <!--origin xyz="0.000299999999999317 0.0160078233491243 -0.0136945669206257" rpy="0 0 0" /-->
+	<origin xyz="0 0 0" rpy="0 0 0" />
         <mass value="0.0104003125914103" />
         <inertia
@@ -228,5 +229,6 @@
       </inertial>
       <visual>
-        <origin xyz="0 0.02 -0.05" rpy="0 0 0" />
+        <!--origin xyz="0 0.02 -0.05" rpy="0 0 0" /-->
+	<origin xyz="0 0 0" rpy="0 0 0" />
         <geometry>
           <mesh filename="package://icl_ur5_setup_description/meshes/robotiq_arg2f_${stroke}_finger_tip.dae" scale="1.0 1.0 1.0"/>
@@ -245,6 +247,6 @@
     <gazebo reference="${prefix}${fingerprefix}_finger_tip">
       <implicitSpringDamper>1</implicitSpringDamper>
-      <mu1>1.0</mu1>
-      <mu2>1.0</mu2>
+      <mu1>100000.0</mu1>
+      <mu2>100000.0</mu2>
       <kp>1000.0</kp>
       <kd>1.0</kd>
@@ -255,8 +257,10 @@
   <xacro:macro name="finger_tip_joint" params="prefix fingerprefix">
     <joint name="${prefix}${fingerprefix}_finger_tip_joint" type="fixed">
-      <origin xyz="0 0.01821998610742 0.0260018192872234" rpy="0 0 0" />
+      <!--origin xyz="0 0.01821998610742 0.0260018192872234" rpy="0 0 0" /-->
+	<origin xyz="0 0.0457554015893473 -0.0272203446692936" rpy="0 0 0" />
       <parent link="${prefix}${fingerprefix}_inner_finger" />
       <child link="${prefix}${fingerprefix}_finger_tip" />
-      <axis xyz="1 0 0" />
+      <!--axis xyz="1 0 0" /-->
+      <axis xyz="0 0 1" />
     </joint>
   </xacro:macro>

File: icl_ur5_setup_description/urdf/sensors/kinect2.gazebo.xacro (robot description, xacro)
@@ -5,5 +5,5 @@
     <sensor type="depth" name="${name}_ir_sensor">
       <always_on>true</always_on>
-      <update_rate>1.0</update_rate>
+      <update_rate>10.0</update_rate>
       <camera>
         <horizontal_fov>${57.0*M_PI/180.0}</horizontal_fov>
@@ -21,5 +21,5 @@
         <baseline>0.2</baseline>
         <alwaysOn>true</alwaysOn>
-        <updateRate>1.0</updateRate>
+        <updateRate>10</updateRate>
         <cameraName>${camera_name}_ir</cameraName>
         <imageTopicName>/${camera_name}/ir/image_raw</imageTopicName>
@@ -31,9 +31,9 @@
         <!--pointCloudCutoff>1.5</pointCloudCutoff-->
         <!--pointCloudCutoffMax>3.0</pointCloudCutoffMax-->
-        <pointCloudCutoff>0.5</pointCloudCutoff>
+        <!--pointCloudCutoff>0.5</pointCloudCutoff-->
         <distortionK1>0.00000001</distortionK1>
         <distortionK2>0.00000001</distortionK2>
         <distortionK3>0.00000001</distortionK3>
-        <distortionT1>0.00000001</distortionT1>a
+        <distortionT1>0.00000001</distortionT1>
         <distortionT2>0.00000001</distortionT2>
         <CxPrime>0</CxPrime>
@@ -51,5 +51,5 @@
     <sensor type="depth" name="${name}_rgb_sensor">
       <always_on>true</always_on>
-      <update_rate>1.0</update_rate>
+      <update_rate>10.0</update_rate>
       <camera>
         <horizontal_fov>${57.0*M_PI/180.0}</horizontal_fov>
@@ -66,5 +66,5 @@
       <plugin name="${link_name}_controller" filename="libgazebo_ros_openni_kinect.so">
         <alwaysOn>true</alwaysOn>
-        <updateRate>1.0</updateRate>
+        <updateRate>10</updateRate>
         <cameraName>${camera_name}_rgb</cameraName>
         <imageTopicName>/${camera_name}/rgb/image_raw</imageTopicName>
@@ -74,5 +74,5 @@
         <pointCloudTopicName>/${camera_name}/depth_registered/points</pointCloudTopicName>
         <frameName>${frame_name}</frameName>
-        <pointCloudCutoff>0.5</pointCloudCutoff>
+        <!--pointCloudCutoff>0.5</pointCloudCutoff-->
         <distortionK1>0.00000001</distortionK1>
         <distortionK2>0.00000001</distortionK2>

File: icl_ur5_setup_description/urdf/sensors/kinect2.urdf.xacro (robot description, xacro)
@@ -2,5 +2,6 @@
 <robot xmlns:xacro="http://wiki.ros.org/xacro">
   <xacro:include filename="$(find icl_ur5_setup_description)/urdf/sensors/kinect2.gazebo.xacro" />
-  <xacro:property name="ir_depth_rgb_offset_y" value="0.01"/> <!-- FIXME: what is this offset? -->
+  <!--xacro:property name="ir_depth_rgb_offset_y" value="0.01"/--> <!-- FIXME: what is this offset? -->
+  <xacro:property name="ir_depth_rgb_offset_y" value="0.0"/>
   <!-- Kinect2 and mount assembly -->
   <xacro:macro name="kinect2_v0" params="name parent *origin">
@@ -73,5 +74,6 @@
     <!-- kinect2 rgb sensor physical attachment -->
     <joint name="${name}_kinect2_rgb_joint" type="fixed">
-      <origin xyz="0 -0.05175 0" rpy="0 0 0"/>
+      <origin xyz="0 0 0" rpy="0 0 0"/>
+      <!--origin xyz="0 -0.05175 0" rpy="0 0 0"/-->
       <parent link="${name}_kinect2_ir_link"/>
       <child link="${name}_kinect2_rgb_link"/>
