Commit message: add calibration model

File: icl_ur5_setup_description/robots/calibration/ur5_robotiq_140_joint_limited.xacro (robot description, xacro)
@@ -50,9 +50,15 @@
       <origin xyz=" 0.0 0.0 0.0" rpy="0.0 0.0 0.0" />
     </joint>
+    <!--link name="${prefix}tool" />
+    <joint name="tool_tip" type="fixed">
+      <parent link= "${prefix}ee_link" />
+      <child link = "${prefix}tool" />
+      <origin xyz=" 0.2 0.0 0.0" rpy="0.0 0.0 0.0" />
+    </joint-->
     <link name="${prefix}tool" />
     <joint name="tool_tip" type="fixed">
       <parent link= "${prefix}ee_link" />
       <child link = "${prefix}tool" />
-      <origin xyz=" 0.2 0.0 0.0" rpy="0.0 0.0 0.0" />
+      <origin xyz="0.234333227426 0.0 0.0" rpy="1.57064 0.0 1.57067" />
     </joint>
   </xacro:macro>

File: icl_ur5_setup_description/urdf/robotiq_arg2f_140_model_macro.xacro (robot description, xacro)
@@ -232,14 +232,14 @@
 	<origin xyz="0 0 0" rpy="0 0 0" />
         <geometry>
-          <mesh filename="package://icl_ur5_setup_description/meshes/robotiq_arg2f_${stroke}_finger_tip.dae" scale="1.0 1.0 1.0"/>
-        </geometry>
-        <material name="">
-          <color rgba="0.1 0.1 0.1 1" />
-        </material>
-      </visual>
-      <collision>
-        <origin xyz="0 0 0" rpy="0 0 0" />
-        <geometry>
-          <mesh filename="package://icl_ur5_setup_description/meshes/robotiq_arg2f_${stroke}_finger_tip.dae" scale="1.0 1.0 1.0"/>
+          <mesh filename="package://icl_ur5_setup_description/meshes/robotiq_arg2f_${stroke}_finger_tip.dae" scale="0.8 0.8 0.8"/>
+        </geometry>
+        <material name="">
+          <color rgba="0.1 0.1 0.1 1" />
+        </material>
+      </visual>
+      <collision>
+        <origin xyz="0 0 0" rpy="0 0 0" />
+        <geometry>
+          <mesh filename="package://icl_ur5_setup_description/meshes/robotiq_arg2f_${stroke}_finger_tip.dae" scale="0.8 0.8 0.8"/>
         </geometry>
       </collision>

File: icl_ur5_setup_description/urdf/sensors/kinect2.gazebo.xacro (robot description, xacro)
@@ -55,5 +55,5 @@
         <horizontal_fov>${57.0*M_PI/180.0}</horizontal_fov>
         <image>
-          <format>B8G8R8</format>
+          <format>R8G8B8</format>
           <width>640</width>
           <height>480</height>
