Commit message: sych repo

File: ur5_gripper_description/robots/ur5_robotiq_140_joint_limited.xacro (robot description, xacro)
@@ -18,9 +18,9 @@
     <xacro:ur5_robot prefix="${prefix}" joint_limited="true"
       shoulder_pan_lower_limit="${-2*pi}" shoulder_pan_upper_limit="${2*pi}"
-      shoulder_lift_lower_limit="${-pi}" shoulder_lift_upper_limit="${pi}"
-      elbow_joint_lower_limit="${-pi}" elbow_joint_upper_limit="${pi}"
-      wrist_1_lower_limit="${-pi}" wrist_1_upper_limit="${pi}"
-      wrist_2_lower_limit="${-pi}" wrist_2_upper_limit="${pi}"
-      wrist_3_lower_limit="${-pi}" wrist_3_upper_limit="${pi}"
+      shoulder_lift_lower_limit="${-2*pi}" shoulder_lift_upper_limit="${2*pi}"
+      elbow_joint_lower_limit="${-2*pi}" elbow_joint_upper_limit="${2*pi}"
+      wrist_1_lower_limit="${-2*pi}" wrist_1_upper_limit="${2*pi}"
+      wrist_2_lower_limit="${-2*pi}" wrist_2_upper_limit="${2*pi}"
+      wrist_3_lower_limit="${-2*pi}" wrist_3_upper_limit="${2*pi}"
     />
     <link name="world" />
@@ -29,9 +29,9 @@
       <child link = "${prefix}base_link" />
       <!--origin xyz="0.0 0.0 0.0" rpy="0.0 0.0 0.0" /-->
-      <origin xyz="0.0 0.0 0.7" rpy="0.0 0.0 0.0" />
+      <origin xyz="0.0 0.0 0.4" rpy="0.0 0.0 0.0" />
     </joint>
     <!--force torque sensor-->
     <xacro:robotiq_fts150 prefix="" parent="ee_link" >
-      <origin xyz="0.009 0 0 " rpy="-${pi/2} 0 -${pi/2}"/>
+      <origin xyz="0.001 0 0 " rpy="-${pi/2} 0 -${pi/2}"/>
     </xacro:robotiq_fts150>
    <!-- gripper -->
@@ -41,33 +41,39 @@
       <child link = "${prefix}robotiq_arg2f_base_link" />
       <!--origin xyz=" 0.0 0.0 0.0" rpy="0.0 0.0 ${pi/2}" /-->
-      <origin xyz=" 0.0 0.0 0.0" rpy="0.0 0.0 ${pi/2}" />
+      <origin xyz=" 0.0 0.0 0.0" rpy="0.0 0.0 0.0" />
     </joint>
+    <!--link name="${prefix}tool" />
+    <joint name="tool_tip" type="fixed">
+      <parent link= "${prefix}ee_link" />
+      <child link = "${prefix}tool" />
+      <origin xyz=" 0.2 0.0 0.0" rpy="0.0 0.0 0.0" />
+    </joint-->
     <link name="${prefix}tool" />
     <joint name="tool_tip" type="fixed">
       <parent link= "${prefix}ee_link" />
       <child link = "${prefix}tool" />
-      <origin xyz=" 0.00 0.0 0.2" rpy="0.0 0.0 0.0" />
+      <origin xyz="0.234333227426 0.0 0.0" rpy="1.57064 0.0 1.57067" />
     </joint>
-    </xacro:macro>
+  </xacro:macro>
   <xacro:ur5_with_gripper_joint_limited prefix=""/>
  <!-- Plugin -->
-  <gazebo>
+  <!--gazebo>
     <plugin name="gazebo_grasp_fix" filename="libgazebo_grasp_fix.so">
       <arm>
-          <arm_name>robot</arm_name>
+          <arm_name>ur5_robot</arm_name>
           <palm_link>wrist_3_link</palm_link>
           <gripper_link>left_inner_finger</gripper_link>
-          <gripper_link>right_inner_finger</gripper_link>
-          <gripper_link>left_inner_knuckle</gripper_link>
-          <gripper_link>right_inner_knuckle</gripper_link>
-      </arm>
+          <gripper_link>right_inner_finger</gripper_link-->
+          <!--gripper_link>left_inner_knuckle</gripper_link>
+          <gripper_link>right_inner_knuckle</gripper_link-->
+      <!--/arm>
       <forces_angle_tolerance>120</forces_angle_tolerance>
       <update_rate>4</update_rate>
       <grip_count_threshold>4</grip_count_threshold>
       <max_grip_count>8</max_grip_count>
-      <release_tolerance>0.05</release_tolerance>
+      <release_tolerance>0.02</release_tolerance>
       <disable_collisions_on_attach>true</disable_collisions_on_attach>
       <contact_topic>__default_topic__</contact_topic>
     </plugin>
-  </gazebo>
+  </gazebo-->
 </robot>

File: ur5_gripper_description/robots/ur5_robotiq_3f_joint_limited.xacro (robot description, xacro)
@@ -4,9 +4,8 @@
   <xacro:include filename="$(find ur_description)/urdf/common.gazebo.xacro" />
   <xacro:include filename="$(find ur_description)/urdf/ur5.urdf.xacro" />
-  <xacro:include filename="$(find ur5_gripper_description)/urdf/robotiq_arg2f_140_model_macro.xacro" />
+  <xacro:include filename="$(find ur5_gripper_description)/urdf/robotiq_3f_hand.urdf.xacro" />
+  <!--xacro:include filename="$(find ur5_gripper_description)/urdf/robotiq_arg2f_140_model_macro.xacro" /-->
   <xacro:include filename="$(find ur5_gripper_description)/urdf/robotiq_fts300.urdf.xacro" />
-  <xacro:include filename="$(find ur5_gripper_description)/urdf/sensors/common.xacro" />
-  <xacro:include filename="$(find ur5_gripper_description)/urdf/sensors/kinect2.urdf.xacro" />
-  <xacro:macro name="ur5_with_gripper_joint_limited" params="prefix">
+  <xacro:macro name="ur5_with_3f_gripper_joint_limited" params="prefix">
     <!-- arm -->
     <!--xacro:ur5_robot prefix="${prefix}" joint_limited="true"
@@ -34,15 +33,17 @@
     </joint>
     <!--force torque sensor-->
-    <xacro:robotiq_fts150 prefix="" parent="ee_link" >
+    <!--xacro:robotiq_fts150 prefix="${prefix}" parent="ee_link" >
       <origin xyz="0.001 0 0 " rpy="-${pi/2} 0 -${pi/2}"/>
-    </xacro:robotiq_fts150>
+    </xacro:robotiq_fts150-->
    <!-- gripper -->
-    <xacro:robotiq_arg2f_140 prefix="${prefix}" />
-    <joint name="ur5_ee_link_gripper_base" type="fixed">
-      <parent link= "${prefix}fts_toolside" />
-      <child link = "${prefix}robotiq_arg2f_base_link" />
+    <xacro:robotiq_hand prefix="${prefix}" parent="ee_link" reflect="1">
+       <origin rpy="0 0 ${-pi/2.0}" xyz="0.051 0 0"/>
+    </xacro:robotiq_hand>
+    <!--joint name="ur5_ee_link_gripper_base" type="fixed">
+      <parent link= "${prefix}fts_toolside" /-->
+      <!--child link = "${prefix}robotiq_arg2f_base_link" /-->
       <!--origin xyz=" 0.0 0.0 0.0" rpy="0.0 0.0 ${pi/2}" /-->
-      <origin xyz=" 0.0 0.0 0.0" rpy="0.0 0.0 0.0" />
-    </joint>
+      <!--origin rpy="0 0 0" xyz="0 0 0" />
+    </joint-->
     <!--link name="${prefix}tool" />
     <joint name="tool_tip" type="fixed">
@@ -51,20 +52,22 @@
       <origin xyz=" 0.2 0.0 0.0" rpy="0.0 0.0 0.0" />
     </joint-->
-    <link name="${prefix}tool" />
+    <!--link name="${prefix}tool" />
     <joint name="tool_tip" type="fixed">
       <parent link= "${prefix}ee_link" />
       <child link = "${prefix}tool" />
       <origin xyz="0.234333227426 0.0 0.0" rpy="1.57064 0.0 1.57067" />
-    </joint>
+    </joint-->
   </xacro:macro>
-    <xacro:kinect2_v0 name="" parent="world" >
-      <!--origin xyz="0.4 0.0 1.2" rpy="0.0 ${pi/2} 0.0" /-->
-      <!--origin xyz="2 0.0 1.3" rpy="0.0 ${pi/3} ${pi}" /-->
-      <!--origin xyz="-1.3 1.3 1.3" rpy="0.0 ${2*pi/9} ${-1*pi/4}" /-->
-      <origin xyz="1.3 -1.3 1.3" rpy="0.0 ${2*pi/9} ${3*pi/4}" />
-    </xacro:kinect2_v0>
-  <xacro:ur5_with_gripper_joint_limited prefix=""/>
+  <xacro:ur5_with_3f_gripper_joint_limited prefix=""/>
+  <gazebo>
+    <!-- plugin for left RobotiQ hand -->
+    <plugin name="robotiq_hand_plugin" filename="libRobotiqHandPlugin.so">
+      <!--side>left</side-->
+      <kp_position>10.0</kp_position>
+      <kd_position>0.5</kd_position>
+    </plugin>
+  </gazebo>
  <!-- Plugin -->
-  <gazebo>
+  <!--gazebo>
     <plugin name="gazebo_grasp_fix" filename="libgazebo_grasp_fix.so">
       <arm>
@@ -72,8 +75,8 @@
           <palm_link>wrist_3_link</palm_link>
           <gripper_link>left_inner_finger</gripper_link>
-          <gripper_link>right_inner_finger</gripper_link>
+          <gripper_link>right_inner_finger</gripper_link-->
           <!--gripper_link>left_inner_knuckle</gripper_link>
           <gripper_link>right_inner_knuckle</gripper_link-->
-      </arm>
+      <!--/arm>
       <forces_angle_tolerance>120</forces_angle_tolerance>
       <update_rate>4</update_rate>
@@ -84,4 +87,4 @@
       <contact_topic>__default_topic__</contact_topic>
     </plugin>
-  </gazebo>
+  </gazebo-->
 </robot>

File: ur5_gripper_description/urdf/robotiq_arg2f_140_model_macro.xacro (robot description, xacro)
@@ -230,16 +230,16 @@
       <visual>
         <!--origin xyz="0 0.02 -0.05" rpy="0 0 0" /-->
-	<origin xyz="0 0 0" rpy="0 0 0" />
-        <geometry>
-          <mesh filename="package://ur5_gripper_description/meshes/robotiq_arg2f_${stroke}_finger_tip.dae" scale="0.8 0.8 0.8"/>
-        </geometry>
-        <material name="">
-          <color rgba="0.1 0.1 0.1 1" />
-        </material>
-      </visual>
-      <collision>
-        <origin xyz="0 0 0" rpy="0 0 0" />
-        <geometry>
-          <mesh filename="package://ur5_gripper_description/meshes/robotiq_arg2f_${stroke}_finger_tip.dae" scale="0.8 0.8 0.8"/>
+	<origin xyz="0 0.01 0" rpy="0 0 0" />
+        <geometry>
+          <mesh filename="package://ur5_gripper_description/meshes/robotiq_arg2f_${stroke}_finger_tip.dae" scale="1 1 1"/>
+        </geometry>
+        <material name="">
+          <color rgba="0.1 0.1 0.1 1" />
+        </material>
+      </visual>
+      <collision>
+        <origin xyz="0 0.01 0" rpy="0 0 0" />
+        <geometry>
+          <mesh filename="package://ur5_gripper_description/meshes/robotiq_arg2f_${stroke}_finger_tip.dae" scale="1 1 1"/>
         </geometry>
       </collision>
